Commit message: add camera

File: description/camera.xacro (robot description, xacro)
@@ -1,17 +1,29 @@
 <?xml version="1.0"?>
 <robot xmlns:xacro="http://www.ros.org/wiki/xacro">
+    <gazebo>
+        <plugin filename="gz-sim-sensors-system" name="gz::sim::systems::Sensors">
+            <render_engine>ogre2</render_engine>
+        </plugin>
+    </gazebo>
     <gazebo reference="camera_sensor_link">
-        <sensor name="camera_sensor" type="camera">
-            <pose> 0 0 0 0 0 0</pose>
+        <sensor name="camera1" type="camera">
+            <pose> 0 0 0 0 0 1.5708</pose>
             <visualize>true</visualize>
-            <update_rate>24</update_rate>
+            <update_rate>30.0</update_rate>
             <camera>
-                <horizontal_fov>1.57080</horizontal_fov>
+                <camera_info_topic>camera1/camera_info</camera_info_topic>
+                <horizontal_fov>1.3962634</horizontal_fov>
                 <image>
+                    <width>640</width>
+                    <height>480</height>
                     <format>R8G8B8</format>
-                    <width>1920</width>
-                    <height>1080</height>
                 </image>
+                <clip>
+                    <near>0.002</near>
+                    <far>300</far>
+                </clip>
             </camera>
+            <topic>camera1/image</topic>
+            <gz_frame_id>camera_link_optical</gz_frame_id>
         </sensor>
     </gazebo>

File: description/car.urdf.xacro (robot description, xacro)
@@ -4,4 +4,4 @@
     <xacro:include filename="gazebo_colors.xacro" />
     <xacro:include filename="ros2_control.xacro" />
-<!--    <xacro:include filename="camera.xacro" />-->
+    <xacro:include filename="camera.xacro" />
 </robot>

File: description/car_core.urdf.xacro (robot description, xacro)
@@ -87,22 +87,5 @@
         </visual>
     </link>
-    <link name="camera_sensor_link">
-        <sensor name="camera_sensor" type="camera">
-            <origin rpy="-1.57080 0.00000 0.00000" xyz="0.00000 0.00000 0.00000"/>
-            <parent link="camera_sensor_link"/>
-            <camera>
-                <image>
-                    <width>1920</width>
-                    <height>1080</height>
-                    <hfov>1.57080</hfov>
-                </image>
-            </camera>
-        </sensor>
-        <inertial>
-            <inertia ixx="0.00001" ixy="0.00000" ixz="0.00000" iyy="0.00001" iyz="0.00000" izz="0.00001"/>
-            <origin rpy="0.00000 0.00000 0.00000" xyz="0.00000 0.00000 0.00000"/>
-            <mass value="0.00001"/>
-        </inertial>
-    </link>
+    <link name="camera_sensor_link"/>
     <link name="rotate">
         <collision name="rotator_collision">

Commit message: add slam

File: description/camera.xacro (robot description, xacro)
@@ -25,5 +25,5 @@
             </camera>
             <topic>camera1/image</topic>
-            <gz_frame_id>camera_link_optical</gz_frame_id>
+            <gz_frame_id>camera_sensor_link</gz_frame_id>
         </sensor>
     </gazebo>

File: description/car.urdf.xacro (robot description, xacro)
@@ -4,4 +4,5 @@
     <xacro:include filename="gazebo_colors.xacro" />
     <xacro:include filename="ros2_control.xacro" />
-    <xacro:include filename="camera.xacro" />
+<!--    <xacro:include filename="camera.xacro" />-->
+    <xacro:include filename="lidar.xacro" />
 </robot>

File: description/car_core.urdf.xacro (robot description, xacro)
@@ -1,53 +1,65 @@
 <robot name="camera_car_simple" version="1.0">
+    <joint name="base_joint" type="fixed">
+        <parent link="base_link"/>
+        <child link="body"/>
+        <origin rpy="0 0 0" xyz="0 0 0"/>
+    </joint>
+    <joint name="base_footprint_joint" type="fixed">
+        <parent link="base_link"/>
+        <child link="base_footprint"/>
+        <origin rpy="0 0 0" xyz="0 0 0"/>
+    </joint>
     <joint name="cam_joint" type="revolute">
-        <limit lower="-3.14000" upper="3.14000" effort="100.00000" velocity="100.00000"/>
-        <origin rpy="0.00000 0.00000 -0.00000" xyz="0.02000 0.00000 0.07000"/>
+        <limit lower="-3.14000" upper="3.14000" effort="100" velocity="100"/>
+        <origin rpy="0 0 -0" xyz="0.02000 0 0.07000"/>
         <parent link="rotate"/>
         <child link="cam"/>
-        <axis xyz="1.00000 0.00000 0.00000"/>
+        <axis xyz="1.00000 0 0"/>
     </joint>
     <joint name="camera_sensor_link_joint" type="fixed">
-        <origin rpy="0.00000 0.00000 -0.00000" xyz="-0.02000 0.03499 -0.00083"/>
+        <origin rpy="0 0 -0" xyz="-0.02000 0.03499 -0.00083"/>
         <parent link="cam"/>
         <child link="camera_sensor_link"/>
     </joint>
     <joint name="rotate_joint" type="revolute">
-        <limit lower="-3.14000" upper="3.14000" effort="100.00000" velocity="100.00000"/>
-        <origin rpy="0.00000 0.00000 -1.57080" xyz="0.00000 0.00000 0.00000"/>
+        <limit lower="-3.14000" upper="3.14000" effort="100" velocity="100"/>
+        <origin rpy="0 0 -1.57080" xyz="0 0 0"/>
         <parent link="body"/>
         <child link="rotate"/>
-        <axis xyz="0.00000 0.00000 1.00000"/>
+        <axis xyz="0 0 1.00000"/>
     </joint>
     <joint name="wheel_bl_joint" type="continuous">
-        <limit lower="0" upper="0" effort="100.00000" velocity="100.00000"/>
-        <origin rpy="0.00000 0.00000 -1.57080" xyz="-0.15500 0.20000 -0.07600"/>
+        <limit lower="0" upper="0" effort="100" velocity="100"/>
+        <origin rpy="0 0 -1.57080" xyz="-0.15500 0.20000 -0.07600"/>
         <parent link="body"/>
         <child link="wheel_bl"/>
-        <axis xyz="-1.00000 0.00000 0.00000"/>
+        <axis xyz="-1.00000 0 0"/>
     </joint>
     <joint name="wheel_br_joint" type="continuous">
-        <limit lower="0" upper="0" effort="100.00000" velocity="100.00000"/>
-        <origin rpy="0.00000 0.00000 -1.57080" xyz="-0.15500 -0.20000 -0.07600"/>
+        <limit lower="0" upper="0" effort="100" velocity="100"/>
+        <origin rpy="0 0 -1.57080" xyz="-0.15500 -0.20000 -0.07600"/>
         <parent link="body"/>
         <child link="wheel_br"/>
-        <axis xyz="-1.00000 0.00000 0.00000"/>
+        <axis xyz="-1.00000 0 0"/>
     </joint>
     <joint name="wheel_fl_joint" type="continuous">
-        <limit lower="0" upper="0" effort="100.00000" velocity="100.00000"/>
-        <origin rpy="0.00000 0.00000 -1.57080" xyz="0.15500 0.20000 -0.07600"/>
+        <limit lower="0" upper="0" effort="100" velocity="100"/>
+        <origin rpy="0 0 -1.57080" xyz="0.15500 0.20000 -0.07600"/>
         <parent link="body"/>
         <child link="wheel_fl"/>
-        <axis xyz="-1.00000 0.00000 0.00000"/>
+        <axis xyz="-1.00000 0 0"/>
     </joint>
     <joint name="wheel_fr_joint" type="continuous">
-        <limit lower="0" upper="0" effort="100.00000" velocity="100.00000"/>
-        <origin rpy="0.00000 0.00000 -1.57080" xyz="0.15500 -0.20000 -0.07600"/>
+        <limit lower="0" upper="0" effort="100" velocity="100"/>
+        <origin rpy="0 0 -1.57080" xyz="0.15500 -0.20000 -0.07600"/>
         <parent link="body"/>
         <child link="wheel_fr"/>
-        <axis xyz="-1.00000 0.00000 0.00000"/>
-    </joint>
+        <axis xyz="-1.00000 0 0"/>
+    </joint>
+    <link name="base_link"/>
+    <link name="base_footprint"/>
     <link name="body">
         <collision name="body_collision">
-            <origin rpy="0.00000 0.00000 -1.57080" xyz="0.00000 0.00000 0.00000"/>
+            <origin rpy="0 0 -1.57080" xyz="0 0 0"/>
             <geometry>
                 <mesh filename="file:///home/yaroslav/ros2_ws/src/camera_car_simple/description/meshes/stl/body-mesh.stl" scale="1.00000 1.00000 1.00000"/>
@@ -55,10 +67,10 @@
         </collision>
         <inertial>
-            <inertia ixx="0.03987" ixy="0.00000" ixz="0.00000" iyy="0.02791" iyz="-0.00000" izz="0.06464"/>
-            <origin rpy="0.00000 0.00000 0.00000" xyz="0.00000 -0.00000 -0.04608"/>
+            <inertia ixx="0.03987" ixy="0" ixz="0" iyy="0.02791" iyz="-0" izz="0.06464"/>
+            <origin rpy="0 0 0" xyz="0 -0 -0.04608"/>
             <mass value="2.80800"/>
         </inertial>
         <visual name="body-obj">
-            <origin rpy="0.00000 0.00000 -1.57080" xyz="0.00000 0.00000 0.00000"/>
+            <origin rpy="0 0 -1.57080" xyz="0 0 0"/>
             <material name="Материал.001"/>
             <geometry>
@@ -69,5 +81,5 @@
     <link name="cam">
         <collision name="cam_collision">
-            <origin rpy="0.00000 0.00000 -0.00000" xyz="-0.02282 0.00074 -0.00002"/>
+            <origin rpy="0 0 -0" xyz="-0.02282 0.00074 -0.00002"/>
             <geometry>
                 <box size="0.04000 0.05486 0.04091"/>
@@ -75,10 +87,10 @@
         </collision>
         <inertial>
-            <inertia ixx="0.00008" ixy="0.00000" ixz="-0.00000" iyy="0.00006" iyz="0.00000" izz="0.00008"/>
-            <origin rpy="0.00000 0.00000 0.00000" xyz="-0.02000 0.00520 -0.00012"/>
+            <inertia ixx="0.00008" ixy="0" ixz="-0" iyy="0.00006" iyz="0" izz="0.00008"/>
+            <origin rpy="0 0 0" xyz="-0.02000 0.00520 -0.00012"/>
             <mass value="0.26000"/>
         </inertial>
         <visual name="cam-obj">
-            <origin rpy="0.00000 0.00000 -0.00000" xyz="0.00000 0.00000 0.00000"/>
+            <origin rpy="0 0 -0" xyz="0 0 0"/>
             <material name="Материал.001"/>
             <geometry>
@@ -90,5 +102,5 @@
     <link name="rotate">
         <collision name="rotator_collision">
-            <origin rpy="0.00000 0.00000 -0.00000" xyz="0.00000 0.00000 0.00000"/>
+            <origin rpy="0 0 -0" xyz="0 0 0"/>
             <geometry>
                 <mesh filename="file:///home/yaroslav/ros2_ws/src/camera_car_simple/description/meshes/stl/rotate-mesh.stl" scale="1.00000 1.00000 1.00000"/>
@@ -96,10 +108,10 @@
         </collision>
         <inertial>
-            <inertia ixx="0.00006" ixy="-0.00000" ixz="-0.00004" iyy="0.00010" iyz="-0.00000" izz="0.00006"/>
-            <origin rpy="0.00000 0.00000 0.00000" xyz="0.02599 -0.00000 0.03366"/>
+            <inertia ixx="0.00006" ixy="-0" ixz="-0.00004" iyy="0.00010" iyz="-0" izz="0.00006"/>
+            <origin rpy="0 0 0" xyz="0.02599 -0 0.03366"/>
             <mass value="0.10400"/>
         </inertial>
         <visual name="rotate-obj">
-            <origin rpy="0.00000 0.00000 -0.00000" xyz="-0.00000 0.00000 0.00000"/>
+            <origin rpy="0 0 -0" xyz="-0 0 0"/>
             <material name="Материал.001"/>
             <geometry>
@@ -110,16 +122,16 @@
     <link name="wheel_bl">
         <collision name="wheel_bl_collision">
-            <origin rpy="0.00000 1.57080 0.00000" xyz="-0.00989 -0.00004 0.00001"/>
-            <geometry>
-                <cylinder radius="0.05449" length="0.03000"/>
-            </geometry>
-        </collision>
-        <inertial>
-            <inertia ixx="0.00043" ixy="-0.00000" ixz="0.00000" iyy="0.00024" iyz="0.00000" izz="0.00024"/>
-            <origin rpy="0.00000 0.00000 0.00000" xyz="-0.01002 -0.00025 0.00007"/>
+            <origin rpy="0 1.57080 0" xyz="-0.00989 -0.00004 0.00001"/>
+            <geometry>
+                <cylinder radius="0.05449" length="0.03000"/>
+            </geometry>
+        </collision>
+        <inertial>
+            <inertia ixx="0.00043" ixy="-0" ixz="0" iyy="0.00024" iyz="0" izz="0.00024"/>
+            <origin rpy="0 0 0" xyz="-0.01002 -0.00025 0.00007"/>
             <mass value="0.31200"/>
         </inertial>
         <visual name="wheel_bl-obj">
-            <origin rpy="0.00000 0.00000 -0.00000" xyz="-0.00000 -0.00000 0.00000"/>
+            <origin rpy="0 0 -0" xyz="-0 -0 0"/>
             <material name="Материал.001"/>
             <geometry>
@@ -130,16 +142,16 @@
     <link name="wheel_br">
         <collision name="wheel_br_collision">
-            <origin rpy="0.00000 1.57080 0.00000" xyz="0.00992 -0.00004 0.00001"/>
-            <geometry>
-                <cylinder radius="0.05449" length="0.03000"/>
-            </geometry>
-        </collision>
-        <inertial>
-            <inertia ixx="0.00043" ixy="0.00000" ixz="-0.00000" iyy="0.00024" iyz="0.00000" izz="0.00024"/>
-            <origin rpy="0.00000 0.00000 0.00000" xyz="0.01002 -0.00025 0.00007"/>
+            <origin rpy="0 1.57080 0" xyz="0.00992 -0.00004 0.00001"/>
+            <geometry>
+                <cylinder radius="0.05449" length="0.03000"/>
+            </geometry>
+        </collision>
+        <inertial>
+            <inertia ixx="0.00043" ixy="0" ixz="-0" iyy="0.00024" iyz="0" izz="0.00024"/>
+            <origin rpy="0 0 0" xyz="0.01002 -0.00025 0.00007"/>
             <mass value="0.31200"/>
         </inertial>
         <visual name="wheel_br-obj">
-            <origin rpy="0.00000 0.00000 -0.00000" xyz="0.00000 -0.00000 0.00000"/>
+            <origin rpy="0 0 -0" xyz="0 -0 0"/>
             <material name="Материал.001"/>
             <geometry>
@@ -150,16 +162,16 @@
     <link name="wheel_fl">
         <collision name="wheel_fl_collision">
-            <origin rpy="0.00000 1.57080 0.00000" xyz="-0.01010 0.00004 0.00001"/>
-            <geometry>
-                <cylinder radius="0.05449" length="0.03000"/>
-            </geometry>
-        </collision>
-        <inertial>
-            <inertia ixx="0.00043" ixy="0.00000" ixz="0.00000" iyy="0.00024" iyz="-0.00000" izz="0.00024"/>
-            <origin rpy="0.00000 0.00000 0.00000" xyz="-0.01002 0.00025 0.00007"/>
+            <origin rpy="0 1.57080 0" xyz="-0.01010 0.00004 0.00001"/>
+            <geometry>
+                <cylinder radius="0.05449" length="0.03000"/>
+            </geometry>
+        </collision>
+        <inertial>
+            <inertia ixx="0.00043" ixy="0" ixz="0" iyy="0.00024" iyz="-0" izz="0.00024"/>
+            <origin rpy="0 0 0" xyz="-0.01002 0.00025 0.00007"/>
             <mass value="0.31200"/>
         </inertial>
         <visual name="wheel_fl-obj">
-            <origin rpy="0.00000 0.00000 -0.00000" xyz="-0.00000 -0.00000 0.00000"/>
+            <origin rpy="0 0 -0" xyz="-0 -0 0"/>
             <material name="Материал.001"/>
             <geometry>
@@ -170,16 +182,16 @@
     <link name="wheel_fr">
         <collision name="wheel_fr_collision">
-            <origin rpy="0.00000 1.57080 0.00000" xyz="0.00999 0.00004 0.00001"/>
-            <geometry>
-                <cylinder radius="0.05449" length="0.03000"/>
-            </geometry>
-        </collision>
-        <inertial>
-            <inertia ixx="0.00043" ixy="-0.00000" ixz="-0.00000" iyy="0.00024" iyz="-0.00000" izz="0.00024"/>
-            <origin rpy="0.00000 0.00000 0.00000" xyz="0.01002 0.00025 0.00007"/>
+            <origin rpy="0 1.57080 0" xyz="0.00999 0.00004 0.00001"/>
+            <geometry>
+                <cylinder radius="0.05449" length="0.03000"/>
+            </geometry>
+        </collision>
+        <inertial>
+            <inertia ixx="0.00043" ixy="-0" ixz="-0" iyy="0.00024" iyz="-0" izz="0.00024"/>
+            <origin rpy="0 0 0" xyz="0.01002 0.00025 0.00007"/>
             <mass value="0.31200"/>
         </inertial>
         <visual name="wheel_fr-obj">
-            <origin rpy="0.00000 0.00000 -0.00000" xyz="0.00000 0.00000 0.00000"/>
+            <origin rpy="0 0 -0" xyz="0 0 0"/>
             <material name="Материал.001"/>
             <geometry>
@@ -189,5 +201,5 @@
     </link>
     <material name="Материал.001">
-        <color rgba="0.00000 0.00000 0.00000 1.00000"/>
+        <color rgba="0 0 0 1.00000"/>
     </material>
 </robot>
